File: aten-kvm-usb-only-adapter.kicad_sch (KiCad schematic)
At the start: 2 parts, among them J1 DE15_Plug_HighDensity_Mountin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, J2 USB_B

Commit message: v03: Use own footprint for male HD15 connector with wider pin spacing
Parts:
- J1: footprint Connector_Dsub:DSUB-15-HD_Male_Horizontal_P2.29x1.98mm_EdgePinOffset3.03mm_Housed_MountingHolesOffset4.94mm -> own:DSUB-15-HD_Male_Horizontal_Assmann_A-HDS15A-KG-TAXB
Changed lines of the file:
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@@
       (effects (font (size 1.27 1.27)))
     )
-    (property "Footprint" "Connector_Dsub:DSUB-15-HD_Male_Horizontal_P2.29x1.98mm_EdgePinOffset3.03mm_Housed_MountingHolesOffset4.94mm" (at 147.32 86.36 0)
+    (property "Footprint" "own:DSUB-15-HD_Male_Horizontal_Assmann_A-HDS15A-KG-TAXB" (at 147.32 86.36 0)
       (effects (font (size 1.27 1.27)) hide)
     )
